Commit message: updated xacro

File: mkz_sensor_kit_description/urdf/sensor_kit.xacro (robot description, xacro)
@@ -12,5 +12,5 @@
   <xacro:arg name="config_dir" default="$(find mkz_sensor_kit_description)/config"/>
   <!-- Load kit-relative calibration -->
-  <xacro:property name="calibration" value="${xacro.load_yaml('$(arg config_dir)/sensor_kit_calibration.yaml')}"/>
+  <xacro:property name="kit_calib" value="${xacro.load_yaml('$(arg config_dir)/sensor_kit_calibration.yaml')}"/>
   <!-- Include your sensor macros -->
   <xacro:include filename="$(find mkz_sensor_kit_description)/urdf/pandar_64.xacro"/>
@@ -39,10 +39,10 @@
                     topic="/pandar_points" hz="10" gpu="$(arg gpu)">
       <origin
-        xyz="${calibration['sensor_kit_base_link']['hesai_lidar']['x']}
-             ${calibration['sensor_kit_base_link']['hesai_lidar']['y']}
-             ${calibration['sensor_kit_base_link']['hesai_lidar']['z']}"
-        rpy="${calibration['sensor_kit_base_link']['hesai_lidar']['roll']}
-             ${calibration['sensor_kit_base_link']['hesai_lidar']['pitch']}
-             ${calibration['sensor_kit_base_link']['hesai_lidar']['yaw']}" />
+        xyz="${kit_calib['sensor_kit_base_link']['hesai_lidar']['x']}
+             ${kit_calib['sensor_kit_base_link']['hesai_lidar']['y']}
+             ${kit_calib['sensor_kit_base_link']['hesai_lidar']['z']}"
+        rpy="${kit_calib['sensor_kit_base_link']['hesai_lidar']['roll']}
+             ${kit_calib['sensor_kit_base_link']['hesai_lidar']['pitch']}
+             ${kit_calib['sensor_kit_base_link']['hesai_lidar']['yaw']}" />
     </xacro:pandar64>
     <!-- IMU: your macro signature requires explicit numeric params -->
@@ -52,10 +52,10 @@
       parent="${sensor_kit_base_link}"
       namespace=""
-      x="${calibration['sensor_kit_base_link']['imu_link']['x']}"
-      y="${calibration['sensor_kit_base_link']['imu_link']['y']}"
-      z="${calibration['sensor_kit_base_link']['imu_link']['z']}"
-      roll="${calibration['sensor_kit_base_link']['imu_link']['roll']}"
-      pitch="${calibration['sensor_kit_base_link']['imu_link']['pitch']}"
-      yaw="${calibration['sensor_kit_base_link']['imu_link']['yaw']}"
+      x="${kit_calib['sensor_kit_base_link']['imu_link']['x']}"
+      y="${kit_calib['sensor_kit_base_link']['imu_link']['y']}"
+      z="${kit_calib['sensor_kit_base_link']['imu_link']['z']}"
+      roll="${kit_calib['sensor_kit_base_link']['imu_link']['roll']}"
+      pitch="${kit_calib['sensor_kit_base_link']['imu_link']['pitch']}"
+      yaw="${kit_calib['sensor_kit_base_link']['imu_link']['yaw']}"
       fps="100"/>
     <!-- GNSS antenna frame (ARP) – frame only -->
@@ -63,10 +63,10 @@
       name="gnss_link"
       parent="${sensor_kit_base_link}"
-      x="${calibration['sensor_kit_base_link']['gnss_link']['x']}"
-      y="${calibration['sensor_kit_base_link']['gnss_link']['y']}"
-      z="${calibration['sensor_kit_base_link']['gnss_link']['z']}"
-      roll="${calibration['sensor_kit_base_link']['gnss_link']['roll']}"
-      pitch="${calibration['sensor_kit_base_link']['gnss_link']['pitch']}"
-      yaw="${calibration['sensor_kit_base_link']['gnss_link']['yaw']}"/>
+      x="${kit_calib['sensor_kit_base_link']['gnss_link']['x']}"
+      y="${kit_calib['sensor_kit_base_link']['gnss_link']['y']}"
+      z="${kit_calib['sensor_kit_base_link']['gnss_link']['z']}"
+      roll="${kit_calib['sensor_kit_base_link']['gnss_link']['roll']}"
+      pitch="${kit_calib['sensor_kit_base_link']['gnss_link']['pitch']}"
+      yaw="${kit_calib['sensor_kit_base_link']['gnss_link']['yaw']}"/>
   </xacro:macro>
 </robot>

File: mkz_sensor_kit_description/urdf/sensors.xacro (robot description, xacro)
@@ -7,14 +7,14 @@
   <!-- Load base_link → sensor_kit_base_link transform -->
   <xacro:arg name="config_dir" default="$(find mkz_sensor_kit_description)/config"/>
-  <xacro:property name="calibration" value="${xacro.load_yaml('$(arg config_dir)/sensors_calibration.yaml')}"/>
+  <xacro:property name="sensors_calib" value="${xacro.load_yaml('$(arg config_dir)/sensors_calibration.yaml')}"/>
   <!-- Bring in the kit macro and instantiate it on base_link -->
   <xacro:include filename="sensor_kit.xacro"/>
   <xacro:sensor_kit_macro
     parent="base_link"
-    x="${calibration['base_link']['sensor_kit_base_link']['x']}"
-    y="${calibration['base_link']['sensor_kit_base_link']['y']}"
-    z="${calibration['base_link']['sensor_kit_base_link']['z']}"
-    roll="${calibration['base_link']['sensor_kit_base_link']['roll']}"
-    pitch="${calibration['base_link']['sensor_kit_base_link']['pitch']}"
-    yaw="${calibration['base_link']['sensor_kit_base_link']['yaw']}" />
+    x="${sensors_calib['base_link']['sensor_kit_base_link']['x']}"
+    y="${sensors_calib['base_link']['sensor_kit_base_link']['y']}"
+    z="${sensors_calib['base_link']['sensor_kit_base_link']['z']}"
+    roll="${sensors_calib['base_link']['sensor_kit_base_link']['roll']}"
+    pitch="${sensors_calib['base_link']['sensor_kit_base_link']['pitch']}"
+    yaw="${sensors_calib['base_link']['sensor_kit_base_link']['yaw']}" />
 </robot>
