Commit message: pandar64.xacro

File: mkz_sensor_kit_description/urdf/pandar_64.xacro (robot description, xacro)
@@ -8,47 +8,42 @@
   -->
   <xacro:macro name="pandar64" params="parent name topic hz gpu *origin">
-    <!-- Base mount joint places _base_link using caller's <origin/> -->
-    <joint name="${name}_base_mount_joint" type="fixed">
+    <!-- Directly mount the LiDAR frame to the parent using caller's <origin/> -->
+    <joint name="${name}_mount_joint" type="fixed">
       <parent link="${parent}"/>
-      <child link="${name}_base_link"/>
+      <child link="${name}"/>
       <xacro:insert_block name="origin"/>
     </joint>
-    <!-- A simple stacked-cylinder visual to represent the sensor body -->
-    <link name="${name}_base_link">
+    <!-- The LiDAR frame used by your driver and TF.
+         All visuals that were previously on ${name}_base_link are now here,
+         so there is no intermediate ${name}_base_link frame. -->
+    <link name="${name}">
+      <!-- A simple stacked-cylinder visual to represent the sensor body -->
       <visual>
-        <geometry><cylinder length="0.030" radius="0.065"/></geometry>
+        <geometry>
+          <cylinder length="0.030" radius="0.065"/>
+        </geometry>
         <origin xyz="0 0 0.015" rpy="0 0 0"/>
-        <material name="dark_gray"><color rgba="0.3 0.3 0.3 1.0"/></material>
+        <material name="dark_gray">
+          <color rgba="0.3 0.3 0.3 1.0"/>
+        </material>
       </visual>
       <visual>
-        <geometry><cylinder length="0.060" radius="0.065"/></geometry>
+        <geometry>
+          <cylinder length="0.060" radius="0.065"/>
+        </geometry>
         <origin xyz="0 0 0.060" rpy="0 0 0"/>
-        <material name="blue"><color rgba="0.0 0.2 1.0 1.0"/></material>
+        <material name="blue">
+          <color rgba="0.0 0.2 1.0 1.0"/>
+        </material>
       </visual>
       <visual>
-        <geometry><cylinder length="0.050" radius="0.065"/></geometry>
+        <geometry>
+          <cylinder length="0.050" radius="0.065"/>
+        </geometry>
         <origin xyz="0 0 0.115" rpy="0 0 0"/>
-        <material name="dark_gray"/>
+        <material name="light_gray">
+          <color rgba="0.8 0.8 0.8 1.0"/>
+        </material>
       </visual>
-      <visual>
-        <geometry><cylinder length="0.030" radius="0.010"/></geometry>
-        <origin xyz="0.0 0.065 0.010" rpy="1.57 0 0"/>
-        <material name="dark_gray"/>
-      </visual>
-      <inertial>
-        <mass value="0.0"/>
-        <origin xyz="0 0 0"/>
-        <inertia ixx="0" ixy="0" ixz="0" iyy="0" iyz="0" izz="0"/>
-      </inertial>
-    </link>
-    <!-- Fixed joint to the scanning frame.
-         The scanning frame name equals ${name}, e.g., "hesai_lidar" -->
-    <joint name="${name}_base_scan_joint" type="fixed">
-      <origin xyz="0 0 0.060" rpy="0 0 0"/>
-      <parent link="${name}_base_link"/>
-      <child link="${name}"/>
-    </joint>
-    <!-- The LiDAR frame used by your driver and TF -->
-    <link name="${name}">
       <inertial>
         <mass value="0.0"/>
